File: hestia-pathfinder.kicad_pcb (KiCad board)
At the start: 2 copper layers, 106 x 52.2 mm, 16 parts, among them SW1 SW_Push, SW2 SW_Push, SW3 SW_Push, SW4 SW_Push, SW5 SW_Push, U1 XIAO-RP2040-DIP

Commit message: Add files via upload
Parts:
- added G***: LOGO, LOGO, F.Cu at (194.1, 109.1)
- added G***: LOGO, LOGO, F.Cu at (133.0, 101.6)
Other:
- board text added: "Made for Pathfinder"
- board text added: "Simon Blinks"
